Commit message: first commit

File: urdfModel/urdf/inspire_hands.urdf (robot description, URDF)
Before this commit: robot inspire_hand_r, 27 links, 26 joints
Links:
- link L_hand_base_link: geometry collision mesh filename=package://urdf_viewer/meshes/L_hand_base_link.STL; visual mesh filename=package://urdf_viewer/meshes/L_hand_base_link.STL
- link L_index_distal: geometry collision mesh filename=package://urdf_viewer/meshes/L_index_distal.STL; visual mesh filename=package://urdf_viewer/meshes/L_index_distal.STL
- link L_index_proximal: geometry collision mesh filename=package://urdf_viewer/meshes/L_index_proximal.STL; visual mesh filename=package://urdf_viewer/meshes/L_index_proximal.STL
- link L_middle_distal: geometry collision mesh filename=package://urdf_viewer/meshes/L_middle_distal.STL; visual mesh filename=package://urdf_viewer/meshes/L_middle_distal.STL
- link L_middle_proximal: geometry collision mesh filename=package://urdf_viewer/meshes/L_middle_proximal.STL; visual mesh filename=package://urdf_viewer/meshes/L_middle_proximal.STL
- link L_pinky_distal: geometry collision mesh filename=package://urdf_viewer/meshes/L_pinky_distal.STL; visual mesh filename=package://urdf_viewer/meshes/L_pinky_distal.STL
- link L_pinky_proximal: geometry collision mesh filename=package://urdf_viewer/meshes/L_pinky_proximal.STL; visual mesh filename=package://urdf_viewer/meshes/L_pinky_proximal.STL
- link L_ring_distal: geometry collision mesh filename=package://urdf_viewer/meshes/L_ring_distal.STL; visual mesh filename=package://urdf_viewer/meshes/L_ring_distal.STL
- link L_ring_proximal: geometry collision mesh filename=package://urdf_viewer/meshes/L_ring_proximal.STL; visual mesh filename=package://urdf_viewer/meshes/L_ring_proximal.STL
- link L_thumb_distal: geometry collision mesh filename=package://urdf_viewer/meshes/L_thumb_distal.STL; visual mesh filename=package://urdf_viewer/meshes/L_thumb_distal.STL
- link L_thumb_intermediate: geometry collision mesh filename=package://urdf_viewer/meshes/L_thumb_intermediate.STL; visual mesh filename=package://urdf_viewer/meshes/L_thumb_intermediate.STL
- link L_thumb_proximal: geometry collision mesh filename=package://urdf_viewer/meshes/L_thumb_proximal.STL; visual mesh filename=package://urdf_viewer/meshes/L_thumb_proximal.STL
- link L_thumb_proximal_base: geometry collision mesh filename=package://urdf_viewer/meshes/L_thumb_proximal_base.STL; visual mesh filename=package://urdf_viewer/meshes/L_thumb_proximal_base.STL
- link R_hand_base_link: geometry collision mesh filename=package://urdf_viewer/meshes/R_hand_base_link.STL; visual mesh filename=package://urdf_viewer/meshes/R_hand_base_link.STL
- link R_index_distal: geometry collision mesh filename=package://urdf_viewer/meshes/R_index_distal.STL; visual mesh filename=package://urdf_viewer/meshes/R_index_distal.STL
- link R_index_proximal: geometry collision mesh filename=package://urdf_viewer/meshes/R_index_proximal.STL; visual mesh filename=package://urdf_viewer/meshes/R_index_proximal.STL
- link R_middle_distal: geometry collision mesh filename=package://urdf_viewer/meshes/R_middle_distal.STL; visual mesh filename=package://urdf_viewer/meshes/R_middle_distal.STL
- link R_middle_proximal: geometry collision mesh filename=package://urdf_viewer/meshes/R_middle_proximal.STL; visual mesh filename=package://urdf_viewer/meshes/R_middle_proximal.STL
- link R_pinky_distal: geometry collision mesh filename=package://urdf_viewer/meshes/R_pinky_distal.STL; visual mesh filename=package://urdf_viewer/meshes/R_pinky_distal.STL
- link R_pinky_proximal: geometry collision mesh filename=package://urdf_viewer/meshes/R_pinky_proximal.STL; visual mesh filename=package://urdf_viewer/meshes/R_pinky_proximal.STL
- link R_ring_distal: geometry collision mesh filename=package://urdf_viewer/meshes/R_ring_distal.STL; visual mesh filename=package://urdf_viewer/meshes/R_ring_distal.STL
- link R_ring_proximal: geometry collision mesh filename=package://urdf_viewer/meshes/R_ring_proximal.STL; visual mesh filename=package://urdf_viewer/meshes/R_ring_proximal.STL
- link R_thumb_distal: geometry collision mesh filename=package://urdf_viewer/meshes/R_thumb_distal.STL; visual mesh filename=package://urdf_viewer/meshes/R_thumb_distal.STL
- link R_thumb_intermediate: geometry collision mesh filename=package://urdf_viewer/meshes/R_thumb_intermediate.STL; visual mesh filename=package://urdf_viewer/meshes/R_thumb_intermediate.STL
- link R_thumb_proximal: geometry collision mesh filename=package://urdf_viewer/meshes/R_thumb_proximal.STL; visual mesh filename=package://urdf_viewer/meshes/R_thumb_proximal.STL
- link R_thumb_proximal_base: geometry collision mesh filename=package://urdf_viewer/meshes/R_thumb_proximal_base.STL; visual mesh filename=package://urdf_viewer/meshes/R_thumb_proximal_base.STL
